Commit message: Latest changes

File: install/my_robot_description/share/my_robot_description/urdf/mobile_base.xacro (robot description, xacro)
@@ -37,5 +37,5 @@
             <collision>
                 <geometry>
-                    <sphere radius="${wheel_radius}"/>
+                    <sphere radius="${wheel_radius}" />
                 </geometry>
                 <origin xyz="0 0 0" rpy="${pi / 2.0} 0 0" />
@@ -57,5 +57,5 @@
         <collision>
             <geometry>
-                <sphere radius="${wheel_radius}"/>
+                <sphere radius="${wheel_radius}" />
             </geometry>
             <origin xyz="0 0 0" rpy="${pi / 2.0} 0 0" />
@@ -65,5 +65,5 @@
         <parent link="base_footprint" />
         <child link="base_link" />
-        <origin xyz="0 0 ${wheel_radius}" rpy="0 0 0"/>
+        <origin xyz="0 0 ${wheel_radius}" rpy="0 0 0" />
     </joint>
     <joint name="base_right_wheel_joint" type="continuous">

File: install/my_robot_description/share/my_robot_description/urdf/mobile_base_gazebo.xacro (robot description, xacro)
@@ -5,22 +5,4 @@
         <mu2 value="0.1" />
     </gazebo>
-    <!-- Diff Drive plugin -->
-    <!-- <gazebo>
-        <plugin name="diff_drive" filename="gz-sim-diff-drive-system">
-            <left_joint>base_left_wheel_joint</left_joint>
-            <right_joint>base_right_wheel_joint</right_joint>
-            <wheel_separation>0.45</wheel_separation>
-            <wheel_radius>0.1</wheel_radius>
-            <frame_id>odom</frame_id>
-            <child_frame_id>base_footprint</child_frame_id>
-        </plugin>
-    </gazebo> -->
-    <!-- Joint State Publisher -->
-    <!-- <gazebo>
-        <plugin name="joint_state_pub" filename="gz-sim-joint-state-publisher-system">
-            <joint_name>base_left_wheel_joint</joint_name>
-            <joint_name>base_right_wheel_joint</joint_name>
-        </plugin>
-    </gazebo> -->
     <gazebo>
         <plugin filename="gz-sim-diff-drive-system"
@@ -36,5 +18,5 @@
     <gazebo>
         <plugin filename="gz-sim-joint-state-publisher-system"
-          name="gz::sim::systems::JointStatePublisher">
+            name="gz::sim::systems::JointStatePublisher">
             <joint_name>base_left_wheel_joint</joint_name>
             <joint_name>base_right_wheel_joint</joint_name>
